File: stm32f103-dev-board.brd (EAGLE design)
At the start: 54.3 x 50.8 mm, 33 parts, among them Q1 8MHz, U1 STM32F103CBT6, U2 LM1117MP-3.3, Y1 32.768kHz

Commit message: v0.2
added led on PC13
added power led
added external power in
Parts:
- added D1, D2: (no value), SparkFun-LED:LED_3MM
- added D3, D4: 1A/40V/500mV, SparkFun-DiscreteSemi:SMA-DIODE
- added J5: (no value), SparkFun-Connectors:1X02
- added R1, R9: 470, rcl:R0805
- moved FRAME1 22.9 mm to (-2.54, -7.62)
- moved X1 6.35 mm to (2.03, 32.8)
- moved R6 4.13 mm to (13.5, 20.8), turned to 270 degrees
- moved C10 3.05 mm to (3.05, 12.2)
- moved C9 3.05 mm to (3.05, 9.65)
- moved R2 2.84 mm to (8.89, 34.3)
- moved R4 2.84 mm to (8.89, 31.8)
- moved F1 1.98 mm to (8.89, 21.3), turned to 180 degrees
- moved C12 1.27 mm to (38.1, 41.9)
- moved C13 1.27 mm to (40.6, 41.9)
- moved C6 1.27 mm to (3.05, 19.1)
- moved C7 1.27 mm to (3.05, 16.5)
- moved Y1 1.02 mm to (39.4, 31.0)
Connections:
- new net N$1: D3.A, X1.VBUS
- new net N$2: D2.A, R9.2
- new net N$3: D1.A, R1.2
- new net N$5: D4.A, J5.2
- net +3V3: now also R1.1
- net +5V: now also D3.C, D4.C; no longer X1.VBUS
- net GND: now also D1.K, D2.K, J5.1
- net PC13: now also R9.1
Routing:
- net GND: track 290.1 -> 305.8 mm
- net N$17: track 9.80 -> 3.86 mm
- net N$1: track 0.00 -> 4.82 mm
- net N$16: track 7.91 -> 3.69 mm
- net +3V3: track 211.2 -> 207.2 mm
- net PC13: track 19.4 -> 22.6 mm
- net N$5: track 0.00 -> 2.74 mm
- net N$2: track 0.00 -> 2.58 mm
- net +5V: track 4.31 -> 6.76 mm
- net PA12-DP: track 17.0 -> 19.3 mm
- net PA11-DM: track 14.1 -> 16.4 mm
- net N$3: track 0.00 -> 2.22 mm
- net N$7: track 10.2 -> 8.33 mm
- net PC15: track 21.8 -> 20.2 mm
- net PC14: track 19.1 -> 17.5 mm
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Other:
- board text added: "- + PWR IN"
- board text added: "Curious Mind"
- board text added: "LED"
- board text added: "PWR"

Commit message: corrected usb pullup
corrected usb pullup
routed swdio (PA13)
Parts:
- J3: device SparkFun-Connectors:1X12 -> SparkFun-Connectors:1X13
- moved C2 5.08 mm to (17.8, 32.5)
- moved R3 4.67 mm to (12.2, 35.8), turned to 90 degrees
- moved R6 3.81 mm to (13.5, 24.6)
- moved J1 3.81 mm to (3.81, 39.4)
- moved R7 3.81 mm to (4.57, 43.2)
Connections:
- net PA14 renamed PA14-SWCLK
- removed net PA13: R3.2, U1.34
- new net PA13-SWDIO: J3.13, U1.34
- net +3V3: now also R3.2
Routing:
- net PA13-SWDIO: track 0.00 -> 33.1 mm
- net +3V3: track 207.2 -> 229.2 mm, vias 0 -> 2
- net GND: track 305.8 -> 295.1 mm
- net PA13: track 9.25 -> 0.00 mm
- net BOOT0: track 42.3 -> 43.2 mm
- net N$4: track 3.60 -> 4.45 mm
Other:
- board text added: "A13 A14 A15 B3 B4 B5 B6 B7 B8 B9 GND 3V3 C13"
- board text removed: "A14 A15 B3 B4 B5 B6 B7 B8 B9 GND 3V3 C13"

Commit message: v0.35 optimization
Parts:
- moved C2 1.80 mm to (19.1, 33.8)
Routing:
- net +3V3: track 229.2 -> 205.2 mm, vias 2 -> 0
- net PA13-SWDIO: track 33.1 -> 31.1 mm, vias 0 -> 2
- net GND: track 295.1 -> 296.0 mm
Changed lines of the file:
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@@
 <attribute name="VALUE" x="4.048" y="10.292" size="1.016" layer="28" rot="MR0"/>
 </element>
-<element name="C2" library="rcl" package="C0805K" value="0.1u" x="17.78" y="32.512" smashed="yes" rot="MR0">
-<attribute name="NAME" x="18.78" y="33.387" size="1.016" layer="26" rot="MR0"/>
-<attribute name="VALUE" x="18.78" y="30.612" size="1.016" layer="28" rot="MR0"/>
+<element name="C2" library="rcl" package="C0805K" value="0.1u" x="19.05" y="33.782" smashed="yes" rot="MR0">
+<attribute name="NAME" x="20.05" y="34.657" size="1.016" layer="26" rot="MR0"/>
+<attribute name="VALUE" x="20.05" y="31.882" size="1.016" layer="28" rot="MR0"/>
 </element>
 <element name="C3" library="rcl" package="C0805K" value="0.1u" x="32.766" y="34.798" smashed="yes" rot="MR90">
@@
 <wire x1="2.136453125" y1="36.934453125" x2="2.286" y2="37.084" width="0.4064" layer="16"/>
 <wire x1="2.136453125" y1="36.934453125" x2="2.032" y2="36.83" width="0.4064" layer="16"/>
-<wire x1="3.81" y1="39.37" x2="1.307640625" y2="39.37" width="0.8128" layer="16"/>
 <wire x1="1.307640625" y1="39.37" x2="1.27" y2="39.332359375" width="0.4064" layer="16"/>
-<wire x1="24.9936" y1="30.2006" x2="20.5994" y2="30.2006" width="0.3556" layer="16"/>
-<wire x1="16.7894" y1="30.2006" x2="16.51" y2="30.48" width="0.4064" layer="16"/>
-<wire x1="16.51" y1="30.48" x2="16.51" y2="32.242" width="0.4064" layer="16"/>
-<wire x1="16.51" y1="32.242" x2="16.78" y2="32.512" width="0.4064" layer="16"/>
-<wire x1="20.5994" y1="30.2006" x2="16.7894" y2="30.2006" width="0.4064" layer="16"/>
-<wire x1="16.78" y1="32.512" x2="16.78" y2="32.75" width="0.4064" layer="16"/>
-<wire x1="16.78" y1="32.75" x2="13.97" y2="35.814" width="0.4064" layer="16"/>
 <wire x1="4.826" y1="35.814" x2="3.81" y2="36.83" width="0.4064" layer="16"/>
 <wire x1="3.81" y1="36.83" x2="2.24090625" y2="36.83" width="0.4064" layer="16"/>
 <wire x1="2.24090625" y1="36.83" x2="2.136453125" y2="36.934453125" width="0.4064" layer="16"/>
 <wire x1="13.97" y1="35.814" x2="4.826" y2="35.814" width="0.4064" layer="16"/>
+<wire x1="24.9936" y1="30.2006" x2="23.1394" y2="30.2006" width="0.3556" layer="16"/>
+<wire x1="23.1394" y1="30.2006" x2="21.59" y2="31.75" width="0.3556" layer="16"/>
+<wire x1="18.034" y1="31.75" x2="13.97" y2="35.814" width="0.4064" layer="16"/>
+<wire x1="18.18354375" y1="31.75" x2="21.59" y2="31.75" width="0.4064" layer="16"/>
+<wire x1="18.18354375" y1="31.75" x2="18.034" y2="31.75" width="0.4064" layer="16"/>
+<wire x1="18.05" y1="33.782" x2="18.05" y2="31.88354375" width="0.4064" layer="16"/>
+<wire x1="18.05" y1="31.88354375" x2="18.18354375" y2="31.75" width="0.4064" layer="16"/>
+<wire x1="3.81" y1="39.37" x2="3.81" y2="38.608" width="0.8128" layer="16"/>
+<wire x1="3.81" y1="38.608" x2="2.136453125" y2="36.934453125" width="0.8128" layer="16"/>
+<wire x1="38.354" y1="43.18" x2="38.1" y2="43.41" width="0" layer="19" extent="16-16"/>
+<wire x1="40.64" y1="43.41" x2="40.624" y2="43.18" width="0" layer="19" extent="16-16"/>
 </signal>
 <signal name="+3V3">
@@
 <wire x1="34.29" y1="34.29" x2="34.29" y2="44.45" width="0.4064" layer="16"/>
 <wire x1="34.29" y1="44.45" x2="34.29" y2="46.99" width="0.6096" layer="16"/>
-<wire x1="24.9936" y1="30.6832" x2="24.13" y2="30.6832" width="0.3556" layer="16"/>
 <wire x1="26.4668" y1="23.7236" x2="26.4668" y2="22.8948" width="0.3556" layer="16"/>
 <wire x1="26.4668" y1="22.8948" x2="25.4" y2="21.828" width="0.3556" layer="16"/>
@@
 <wire x1="31.9532" y1="30.6832" x2="31.9532" y2="32.1564" width="0.3556" layer="16"/>
 <wire x1="31.9532" y1="30.6832" x2="29.21" y2="27.94" width="0.4064" layer="16"/>
-<via x="12.446" y="21.112403125" extent="1-16" drill="1"/>
-<wire x1="12.446" y1="21.112403125" x2="12.446" y2="39.116" width="0.6096" layer="1"/>
-<via x="12.446" y="39.116" extent="1-16" drill="1"/>
-<wire x1="12.192" y1="39.37" x2="8.89" y2="39.37" width="0.6096" layer="16"/>
-<wire x1="12.192" y1="39.37" x2="12.446" y2="39.116" width="0.6096" layer="16"/>
-<wire x1="12.192" y1="37.236" x2="12.192" y2="39.37" width="0.6096" layer="16"/>
-<wire x1="12.954" y1="39.116" x2="12.446" y2="39.116" width="0.6096" layer="16"/>
-<wire x1="18.6191" y1="33.909" x2="18.161" y2="33.909" width="0.4064" layer="16"/>
-<wire x1="21.1456" y1="33.909" x2="18.6191" y2="33.909" width="0.4064" layer="16"/>
-<wire x1="18.161" y1="33.909" x2="12.954" y2="39.116" width="0.4064" layer="16"/>
-<wire x1="18.78" y1="32.512" x2="18.78" y2="33.7481" width="0.4064" layer="16"/>
-<wire x1="18.78" y1="33.7481" x2="18.6191" y2="33.909" width="0.4064" layer="16"/>
-<wire x1="24.13" y1="30.6832" x2="24.13" y2="30.9246" width="0.3556" layer="16"/>
-<wire x1="24.13" y1="30.9246" x2="21.1456" y2="33.909" width="0.4064" layer="16"/>
-<wire x1="13.462" y1="21.07748125" x2="13.462" y2="23.688" width="0.4064" layer="16"/>
-<wire x1="13.462" y1="21.07748125" x2="13.462" y2="16.6116" width="0.4064" layer="16"/>
-<wire x1="13.462" y1="16.6116" x2="13.3604" y2="16.51" width="0.4064" layer="16"/>
-<wire x1="12.446" y1="21.112403125" x2="13.427078125" y2="21.112403125" width="0.6096" layer="16"/>
-<wire x1="13.427078125" y1="21.112403125" x2="13.462" y2="21.07748125" width="0.4064" layer="16"/>
+<wire x1="24.9936" y1="30.6832" x2="23.9358375" y2="30.6832" width="0.3556" layer="16"/>
+<wire x1="23.9358375" y1="30.6832" x2="23.9268" y2="30.6832" width="0.3556" layer="16"/>
+<wire x1="24.9936" y1="30.6832" x2="26.4668" y2="30.6832" width="0.3556" layer="16"/>
+<wire x1="26.4668" y1="30.6832" x2="29.21" y2="27.94" width="0.4064" layer="16"/>
+<wire x1="22.191125" y1="32.4279125" x2="23.9358375" y2="30.6832" width="0.3556" layer="16"/>
+<wire x1="22.191125" y1="32.4279125" x2="22.1070375" y2="32.512" width="0.3556" layer="16"/>
+<wire x1="8.89" y1="39.37" x2="10.058" y2="39.37" width="0.4064" layer="16"/>
+<wire x1="10.058" y1="39.37" x2="12.192" y2="37.236" width="0.4064" layer="16"/>
+<wire x1="20.05" y1="34.56" x2="20.05" y2="33.782" width="0.4064" layer="16"/>
+<wire x1="17.374" y1="37.236" x2="20.05" y2="34.56" width="0.4064" layer="16"/>
+<wire x1="12.192" y1="37.236" x2="17.374" y2="37.236" width="0.4064" layer="16"/>
+<wire x1="20.05" y1="33.782" x2="20.8370375" y2="33.782" width="0.4064" layer="16"/>
+<wire x1="20.8370375" y1="33.782" x2="22.191125" y2="32.4279125" width="0.4064" layer="16"/>
+<wire x1="13.3604" y1="16.51" x2="13.462" y2="23.688" width="0" layer="19" extent="16-16"/>
 </signal>
 <signal name="N$7">
@@
 <contactref element="U1" pad="34"/>
 <contactref element="J3" pad="13"/>
-<wire x1="26.67" y1="29.6926" x2="24.9936" y2="29.6926" width="0.3556" layer="16"/>
-<wire x1="26.67" y1="29.6926" x2="26.67" y2="30.48" width="0.3556" layer="16"/>
-<wire x1="26.67" y1="30.48" x2="25.4" y2="31.75" width="0.3556" layer="16"/>
-<wire x1="25.4" y1="34.798" x2="25.4" y2="31.75" width="0.3556" layer="16"/>
-<wire x1="24.9936" y1="29.6926" x2="24.13" y2="29.6926" width="0.3556" layer="16"/>
-<wire x1="9.33135" y1="44.67814375" x2="19.046825" y2="34.798" width="0.4064" layer="16"/>
-<wire x1="19.046825" y1="34.798" x2="25.4" y2="34.798" width="0.4064" layer="16"/>
 <wire x1="6.35" y1="46.99" x2="6.35" y2="45.72" width="0.6096" layer="16"/>
-<wire x1="6.35" y1="45.72" x2="7.39185625" y2="44.67814375" width="0.4064" layer="16"/>
-<wire x1="7.39185625" y1="44.67814375" x2="9.33135" y2="44.67814375" width="0.4064" layer="16"/>
+<wire x1="6.35" y1="45.72" x2="7.39185625" y2="44.67814375" width="0.6096" layer="16"/>
+<wire x1="7.39185625" y1="44.67814375" x2="8.89" y2="44.67814375" width="0.6096" layer="16"/>
+<wire x1="8.89" y1="44.67814375" x2="9.33135" y2="44.67814375" width="0" layer="19" extent="1-16"/>
+<wire x1="17.78" y1="29.6926" x2="24.9936" y2="29.6926" width="0.3556" layer="16"/>
+<via x="14.732" y="32.004" extent="1-16" drill="1"/>
+<wire x1="14.732" y1="32.004" x2="16.256" y2="32.004" width="0.6096" layer="16"/>
+<wire x1="16.256" y1="32.004" x2="17.78" y2="30.48" width="0.6096" layer="16"/>
+<wire x1="17.78" y1="29.764865625" x2="17.78" y2="30.48" width="0.4064" layer="16"/>
+<wire x1="17.78" y1="29.764865625" x2="17.826865625" y2="29.718" width="0.4064" layer="16"/>
+<wire x1="17.78" y1="29.6926" x2="17.78" y2="29.764865625" width="0.3556" layer="16"/>
+<wire x1="14.732" y1="32.004" x2="14.732" y2="38.735" width="0.4064" layer="1"/>
+<via x="14.732" y="38.735" extent="1-16" drill="1"/>
+<wire x1="8.89" y1="44.67814375" x2="8.89" y2="44.577" width="0.4064" layer="16"/>
+<wire x1="8.89" y1="44.577" x2="14.732" y2="38.735" width="0.6096" layer="16"/>
 </signal>
 <signal name="PA12-DP">
